File: escon-carrier-board/escon-carrier-board.kicad_pcb (KiCad board)
At the start: 2 copper layers, 35.6 x 26.7 mm, 3 parts, among them J1 Conn_01x06

Commit message: V.1.0
Parts:
- added G***: LOGO, BohleBots:logo_klein, F.Cu at (26.5, 17.0)
- added H1: MountingHole, MountingHole:MountingHole_2.2mm_M2, F.Cu at (33.0, 7.00)
- added H2: MountingHole, MountingHole:MountingHole_2.2mm_M2, F.Cu at (3.00, 7.00)
- moved JP1 5.41 mm to (25.0, 10.5)
Routing:
- net Net-(ESCON1-+5V): track 23.2 -> 15.5 mm
- net Net-(ESCON1-H1): track 12.4 -> 19.9 mm
- net Net-(J1-Pin_6): track 30.3 -> 25.0 mm
- net Net-(ESCON1-VCC): track 33.5 -> 37.9 mm
- net Net-(ESCON1-M1): track 15.6 -> 12.3 mm
- net Net-(ESCON1-M2): track 15.2 -> 12.1 mm
- net Net-(ESCON1-M3): track 14.5 -> 11.9 mm
- net Net-(ESCON1-H3): track 6.91 -> 9.35 mm
- net Net-(ESCON1-H2): track 7.13 -> 9.13 mm
Other:
- board text added: "ESCON Module 24/2 Carrier Board"
- board text added: "GND D1 D2 D3 D4 VCC"
- board text added: "M1 M2 M3 GND H2 H3 H1 5V"

Commit message: V2.0
Parts:
- moved J1 6.18 mm to (5.83, 16.3)
- moved G*** 1.00 mm to (27.5, 17.0)
Routing:
- net Net-(ESCON1-D4): track 2.16 -> 8.35 mm
- net Net-(ESCON1-D2): track 2.16 -> 8.35 mm
- net Net-(ESCON1-D3): track 2.16 -> 8.35 mm
- net Net-(ESCON1-D1): track 2.16 -> 8.35 mm
- net Net-(ESCON1-VCC): track 37.9 -> 35.3 mm
Changed lines of the file:
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@@
 	(footprint "BohleBots:logo_klein"
 		(layer "F.Cu")
-		(at 26.5 17)
+		(at 27.5 17)
 		(property "Reference" "G***"
 			(at 5.5 14.5 0)
@@
 		(tags "connector JST PH side entry")
 		(property "Reference" "JP1"
-			(at 7 2.9 360)
+			(at 7 2.9 0)
 			(layer "B.SilkS")
 			(hide yes)
@@
 		)
 		(property "Value" "B8B-PH-K"
-			(at 7 -4 360)
+			(at 7 -4 0)
 			(layer "B.Fab")
 			(effects
@@
 		)
 		(fp_text user "${REFERENCE}"
-			(at 7 -1.5 360)
+			(at 7 -1.5 0)
 			(layer "B.Fab")
 			(effects
@@
 	(footprint "Connector_PinHeader_2.54mm:PinHeader_1x06_P2.54mm_Horizontal"
 		(layer "B.Cu")
-		(at 5.8 22.5 -90)
+		(at 5.826498 16.324083 -90)
 		(descr "Through hole angled pin header, 1x06, 2.54mm pitch, 6mm pin length, single row")
 		(tags "Through hole angled pin header THT 1x06 2.54mm single row")
 		(property "Reference" "J1"
-			(at 4.385 2.27 90)
+			(at 2.675917 2.826498 180)
 			(layer "B.SilkS")
+			(hide yes)
 			(effects
 				(font
@@
 	)
 	(gr_text "GND D1 D2 D3 D4 VCC\n"
-		(at 20.5 21 0)
+		(at 21 15 0)
 		(layer "B.SilkS")
 		(effects
@@
 	)
 	(gr_text "M1 M2 M3 GND H2 H3 H1 5V\n"
-		(at 27 15.5 -0)
+		(at 27.5 7.5 -0)
 		(layer "B.SilkS")
 		(effects
@@
 	)
 	(gr_text "ESCON Module 24/2\nCarrier Board\n"
-		(at 1 18.5 0)
+		(at 1 22 0)
 		(layer "F.SilkS")
 		(effects
@@
 	)
 	(segment
-		(start 10.88 22.5)
-		(end 10.88 24.66)
+		(start 10.88 16.350581)
+		(end 10.906498 16.324083)
+		(width 1.2)
+		(layer "F.Cu")
+		(net 1)
+	)
+	(segment
+		(start 10.88 24.66)
+		(end 10.88 16.350581)
 		(width 1.2)
 		(layer "F.Cu")
@@
 	)
 	(segment
-		(start 5.8 22.140862)
-		(end 9.440862 18.5)
+		(start 28.5 11)
+		(end 25.5 14)
 		(width 2)
 		(layer "F.Cu")
@@
 	(segment
 		(start 28.5 5.348)
-		(end 26.12 2.968)
+		(end 28.5 11)
 		(width 2)
 		(layer "F.Cu")
@@
 	)
 	(segment
-		(start 5.8 22.5)
-		(end 5.8 22.140862)
+		(start 25.5 14)
+		(end 7.791443 14)
 		(width 2)
 		(layer "F.Cu")
@@
 	)
 	(segment
-		(start 28.5 11)
-		(end 28.5 5.348)
+		(start 26.12 1.8)
+		(end 26.12 2.968)
 		(width 2)
 		(layer "F.Cu")
@@
 	)
 	(segment
-		(start 21 18.5)
-		(end 28.5 11)
+		(start 7.791443 14)
+		(end 5.826498 15.964945)
 		(width 2)
 		(layer "F.Cu")
@@
 	)
 	(segment
-		(start 9.440862 18.5)
-		(end 21 18.5)
+		(start 5.826498 15.964945)
+		(end 5.826498 16.324083)
 		(width 2)
 		(layer "F.Cu")
@@
 	(segment
 		(start 26.12 2.968)
-		(end 26.12 1.8)
+		(end 28.5 5.348)
 		(width 2)
 		(layer "F.Cu")
@@
 	)
 	(segment
-		(start 8.34 22.5)
+		(start 8.366498 24.633502)
 		(end 8.34 24.66)
 		(width 1.2)
@@
 	)
 	(segment
-		(start 18.5 22.5)
+		(start 8.366498 16.324083)
+		(end 8.366498 24.633502)
+		(width 1.2)
+		(layer "F.Cu")
+		(net 3)
+	)
+	(segment
+		(start 18.526498 24.633502)
 		(end 18.5 24.66)
 		(width 1.2)
@@
 	)
 	(segment
-		(start 19 9)
-		(end 19 10.5)
+		(start 18.526498 16.324083)
+		(end 18.526498 24.633502)
 		(width 1.2)
-		(layer "B.Cu")
+		(layer "F.Cu")
 		(net 4)
 	)
 	(segment
 		(start 19 10.5)
-		(end 19 22)
+		(end 19 15.850581)
 		(width 1.2)
 		(layer "B.Cu")
@@
 	)
 	(segment
-		(start 23.58 1.8)
-		(end 23.58 4.42)
+		(start 19 9)
+		(end 19 10.5)
 		(width 1.2)
 		(layer "B.Cu")
@@
 	)
 	(segment
-		(start 19 22)
-		(end 18.5 22.5)
+		(start 23.58 1.8)
+		(end 23.58 4.42)
 		(width 1.2)
 		(layer "B.Cu")
@@
 	)
 	(segment
-		(start 15.96 22.5)
+		(start 19 15.850581)
+		(end 18.526498 16.324083)
+		(width 1.2)
+		(layer "B.Cu")
+		(net 4)
+	)
+	(segment
+		(start 15.986498 24.633502)
 		(end 15.96 24.66)
 		(width 1.2)
@@
 	)
 	(segment
-		(start 13.42 22.5)
+		(start 15.986498 16.324083)
+		(end 15.986498 24.633502)
+		(width 1.2)
+		(layer "F.Cu")
+		(net 5)
+	)
+	(segment
+		(start 13.446498 16.324083)
+		(end 13.446498 24.633502)
+		(width 1.2)
+		(layer "F.Cu")
+		(net 6)
+	)
+	(segment
+		(start 13.446498 24.633502)
 		(end 13.42 24.66)
 		(width 1.2)

Commit message: V3.0
Connections:
- net Net-(J1-Pin_6) renamed GND
Routing:
- added copper zone on B.Cu, net GND
- added copper zone on F.Cu, net GND
Changed lines of the file:
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@@
 	(net 2 "Net-(ESCON1-VCC)")
 	(net 3 "Net-(ESCON1-D4)")
-	(net 4 "Net-(J1-Pin_6)")
+	(net 4 "GND")
 	(net 5 "Net-(ESCON1-D1)")
 	(net 6 "Net-(ESCON1-D2)")
@@
 		(sheetname "Root")
 		(sheetfile "escon-carrier-board.kicad_sch")
-		(fp_line
-			(start -18.415 -14.605)
-			(end -18.415 12.065)
-			(stroke
-				(width 0.127)
-				(type solid)
-			)
-			(layer "F.SilkS")
-		)
-		(fp_line
-			(start -18.415 12.065)
-			(end 17.145 12.065)
-			(stroke
-				(width 0.127)
-				(type solid)
-			)
-			(layer "F.SilkS")
-		)
-		(fp_line
-			(start 17.145 -14.605)
-			(end -18.415 -14.605)
-			(stroke
-				(width 0.127)
-				(type solid)
-			)
-			(layer "F.SilkS")
-		)
-		(fp_line
-			(start 17.145 12.065)
-			(end 17.145 -14.605)
-			(stroke
-				(width 0.127)
-				(type solid)
-			)
-			(layer "F.SilkS")
-		)
 		(pad "P1" thru_hole rect
 			(at 15.24 -12.7)
@@
 			(layers "*.Cu" "*.Mask")
 			(remove_unused_layers no)
-			(net 4 "Net-(J1-Pin_6)")
+			(net 4 "GND")
 			(pinfunction "GND")
 			(pintype "bidirectional")
@@
 			(layers "*.Cu" "*.Mask")
 			(remove_unused_layers no)
-			(net 4 "Net-(J1-Pin_6)")
+			(net 4 "GND")
 			(pinfunction "GND")
 			(pintype "bidirectional")
@@
 			(layers "*.Cu" "*.Mask")
 			(remove_unused_layers no)
-			(net 4 "Net-(J1-Pin_6)")
+			(net 4 "GND")
 			(pinfunction "4")
 			(pintype "passive")
@@
 			(layers "*.Cu" "*.Mask")
 			(remove_unused_layers no)
-			(net 4 "Net-(J1-Pin_6)")
+			(net 4 "GND")
 			(pinfunction "Pin_6")
 			(pintype "passive")
@@
 		(net 13)
 	)
+	(zone
+		(net 4)
+		(net_name "GND")
+		(layers "F&B.Cu")
+		(hatch edge 0.5)
+		(connect_pads
+			(clearance 0.5)
+		)
+		(min_thickness 0.25)
+		(filled_areas_thickness no)
+		(fill yes
+			(thermal_gap 0.5)
+			(thermal_bridge_width 0.5)
+		)
+		(polygon
+			(pts
+				(xy -3 -2.4) (xy 38.4 -2.4) (xy 38.4 29.8) (xy -3 29.8)
+			)
+		)
+	)
 )

Commit message: V4.0
Routing:
- net GND: track 25.0 -> 0.00 mm
- net Net-(ESCON1-H1): track 19.9 -> 16.7 mm
- net Net-(ESCON1-+5V): track 15.5 -> 14.4 mm

Commit message: V5.0
Parts:
- added G***: LOGO, BohleBots:logo_klein, B.Cu at (27.2, 19.5)
- added H3: MountingHole, MountingHole:MountingHole_2.2mm_M2, F.Cu at (2.00, 13.5)
- added H4: MountingHole, MountingHole:MountingHole_2.2mm_M2, F.Cu at (34.0, 13.5)
- moved G*** 2.51 mm to (27.2, 19.5)
- moved H1 1.00 mm to (34.0, 7.00)
- moved H2 1.00 mm to (2.00, 7.00)
- moved ESCON1 0.71 mm to (18.2, 15.1)
- moved JP1 0.71 mm to (24.7, 11.1)
- moved J1 0.37 mm to (5.53, 16.5)
Routing:
- net GND: track 0.00 -> 25.0 mm
- net Net-(ESCON1-H1): track 16.7 -> 17.3 mm
Other:
- board size 35.6 x 26.7 mm -> 36 x 27 mm

Commit message: Changed to micromatch 10 pole connector
Parts:
- removed JP1: B8B-PH-K, Connector_JST:JST_PH_B8B-PH-K_1x08_P2.00mm_Vertical
- added X1: ~, BohleBots:MICROMATCH-10, B.Cu at (22.0, 10.0)
Routing:
- net Net-(ESCON1-H1): track 17.3 -> 5.57 mm
- net Net-(ESCON1-+5V): track 14.4 -> 7.61 mm
- net Net-(ESCON1-VCC): track 35.3 -> 41.4 mm
- net Net-(ESCON1-M1): track 12.3 -> 17.9 mm
- net Net-(ESCON1-H2): track 9.13 -> 13.3 mm
- net Net-(ESCON1-M2): track 12.1 -> 8.80 mm
- net Net-(ESCON1-H3): track 9.35 -> 8.58 mm
Other:
- board text added: "X M2 GND H3 H1"
- board text added: "X M3 M1 +5V H2"
- board text removed: "M1 M2 M3 GND H2 H3 H1 5V"

Commit message: Gerber Files
Parts:
- removed H1, H2, H3, H4: MountingHole, MountingHole:MountingHole_2.2mm_M2
- moved G*** 0.40 mm to (27.3, 19.9) (x2)
Routing:
- net GND: track 25.0 -> 5.61 mm
Other:
- board size 36 x 27 mm -> 34 x 27 mm
